File: INPUTS.kicad_sch (KiCad schematic)
At the start: 54 parts, among them J6 LED_IN_CONN., J7 LED_IN_CONN., U10 EL817, U11 EL817, U12 EL817, U13 EL817, U14 EL817, U15 EL817, U16 EL817, U7 EL817, U8 EL817, U9 EL817

Commit message: Specefies which section is complete and incomplete
Connections:
- net COMMON renamed COMMON_IN
Changed lines of the file:
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@@
 	(text "INPUT LED"
 		(exclude_from_sim no)
-		(at 33.274 132.842 0)
+		(at 33.274 136.144 0)
 		(effects
 			(font
@@
 	(wire
 		(pts
-			(xy 31.75 118.11) (xy 31.75 128.27)
+			(xy 31.75 118.11) (xy 31.75 130.81)
 		)
 		(stroke
@@
 	(wire
 		(pts
-			(xy 41.91 118.11) (xy 41.91 128.27)
+			(xy 41.91 118.11) (xy 41.91 130.81)
 		)
 		(stroke
@@
 	(wire
 		(pts
-			(xy 46.99 118.11) (xy 46.99 128.27)
+			(xy 46.99 118.11) (xy 46.99 130.81)
 		)
 		(stroke
@@
 	(wire
 		(pts
-			(xy 21.59 118.11) (xy 21.59 128.27)
+			(xy 21.59 118.11) (xy 21.59 130.81)
 		)
 		(stroke
@@
 	(wire
 		(pts
-			(xy 29.21 118.11) (xy 29.21 128.27)
+			(xy 29.21 118.11) (xy 29.21 130.81)
 		)
 		(stroke
@@
 	(wire
 		(pts
-			(xy 44.45 118.11) (xy 44.45 128.27)
+			(xy 44.45 118.11) (xy 44.45 130.81)
 		)
 		(stroke
@@
 	(wire
 		(pts
-			(xy 24.13 118.11) (xy 24.13 128.27)
+			(xy 24.13 118.11) (xy 24.13 130.81)
 		)
 		(stroke
@@
 	(wire
 		(pts
-			(xy 26.67 118.11) (xy 26.67 128.27)
+			(xy 26.67 118.11) (xy 26.67 130.81)
 		)
 		(stroke
@@
 	(wire
 		(pts
-			(xy 39.37 118.11) (xy 39.37 128.27)
+			(xy 39.37 118.11) (xy 39.37 130.81)
 		)
 		(stroke
@@
 	(wire
 		(pts
-			(xy 34.29 118.11) (xy 34.29 128.27)
+			(xy 34.29 118.11) (xy 34.29 130.81)
 		)
 		(stroke
@@
 	(wire
 		(pts
-			(xy 36.83 118.11) (xy 36.83 128.27)
+			(xy 36.83 118.11) (xy 36.83 130.81)
 		)
 		(stroke
@@
 	)
 	(label "LED_IN9"
-		(at 44.45 128.27 90)
+		(at 44.45 130.81 90)
 		(effects
 			(font
@@
 	)
 	(label "LED_IN4"
-		(at 31.75 128.27 90)
+		(at 31.75 130.81 90)
 		(effects
 			(font
@@
 	)
 	(label "LED_IN8"
-		(at 41.91 128.27 90)
+		(at 41.91 130.81 90)
 		(effects
 			(font
@@
 	)
 	(label "LED_IN0"
-		(at 21.59 128.27 90)
+		(at 21.59 130.81 90)
 		(effects
 			(font
@@
 	)
 	(label "LED_IN2"
-		(at 26.67 128.27 90)
+		(at 26.67 130.81 90)
 		(effects
 			(font
@@
 		)
 	)
-	(label "COMMON"
+	(label "COMMON_IN"
 		(at 46.99 105.41 180)
 		(effects
@@
 		)
 	)
-	(label "COMMON"
-		(at 46.99 128.27 90)
+	(label "COMMON_IN"
+		(at 46.99 130.81 90)
 		(effects
 			(font
@@
 	)
 	(label "LED_IN5"
-		(at 34.29 128.27 90)
+		(at 34.29 130.81 90)
 		(effects
 			(font
@@
 	)
 	(label "LED_IN7"
-		(at 39.37 128.27 90)
+		(at 39.37 130.81 90)
 		(effects
 			(font
@@
 	)
 	(label "LED_IN6"
-		(at 36.83 128.27 90)
+		(at 36.83 130.81 90)
 		(effects
 			(font
@@
 	)
 	(label "LED_IN1"
-		(at 24.13 128.27 90)
+		(at 24.13 130.81 90)
 		(effects
 			(font
@@
 	)
 	(label "LED_IN3"
-		(at 29.21 128.27 90)
+		(at 29.21 130.81 90)
 		(effects
 			(font
@@
 		)
 	)
-	(hierarchical_label "COMMON"
+	(hierarchical_label "COMMON_IN"
 		(shape input)
 		(at 85.09 125.73 270)

Commit message: INPUT, PC output resistor size changed from 805 to 603
Parts:
- R31, R43, R46, R47, R52, R53, R54, R55, R58, R59: footprint Resistor_SMD:R_0805_2012Metric_Pad1.20x1.40mm_HandSolder -> Resistor_SMD:R_0603_1608Metric_Pad0.98x0.95mm_HandSolder
Changed lines of the file:
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@@
 			)
 		)
-		(property "Footprint" "Resistor_SMD:R_0805_2012Metric_Pad1.20x1.40mm_HandSolder"
+		(property "Footprint" "Resistor_SMD:R_0603_1608Metric_Pad0.98x0.95mm_HandSolder"
 			(at 151.384 49.276 90)
 			(hide yes)
@@
 			)
 		)
-		(property "Footprint" "Resistor_SMD:R_0805_2012Metric_Pad1.20x1.40mm_HandSolder"
+		(property "Footprint" "Resistor_SMD:R_0603_1608Metric_Pad0.98x0.95mm_HandSolder"
 			(at 151.384 63.246 90)
 			(hide yes)
@@
 			)
 		)
-		(property "Footprint" "Resistor_SMD:R_0805_2012Metric_Pad1.20x1.40mm_HandSolder"
+		(property "Footprint" "Resistor_SMD:R_0603_1608Metric_Pad0.98x0.95mm_HandSolder"
 			(at 151.384 91.186 90)
 			(hide yes)
@@
 			)
 		)
-		(property "Footprint" "Resistor_SMD:R_0805_2012Metric_Pad1.20x1.40mm_HandSolder"
+		(property "Footprint" "Resistor_SMD:R_0603_1608Metric_Pad0.98x0.95mm_HandSolder"
 			(at 151.384 119.126 90)
 			(hide yes)
@@
 			)
 		)
-		(property "Footprint" "Resistor_SMD:R_0805_2012Metric_Pad1.20x1.40mm_HandSolder"
+		(property "Footprint" "Resistor_SMD:R_0603_1608Metric_Pad0.98x0.95mm_HandSolder"
 			(at 151.384 147.066 90)
 			(hide yes)
@@
 			)
 		)
-		(property "Footprint" "Resistor_SMD:R_0805_2012Metric_Pad1.20x1.40mm_HandSolder"
+		(property "Footprint" "Resistor_SMD:R_0603_1608Metric_Pad0.98x0.95mm_HandSolder"
 			(at 151.384 133.096 90)
 			(hide yes)
@@
 			)
 		)
-		(property "Footprint" "Resistor_SMD:R_0805_2012Metric_Pad1.20x1.40mm_HandSolder"
+		(property "Footprint" "Resistor_SMD:R_0603_1608Metric_Pad0.98x0.95mm_HandSolder"
 			(at 151.384 77.216 90)
 			(hide yes)
@@
 			)
 		)
-		(property "Footprint" "Resistor_SMD:R_0805_2012Metric_Pad1.20x1.40mm_HandSolder"
+		(property "Footprint" "Resistor_SMD:R_0603_1608Metric_Pad0.98x0.95mm_HandSolder"
 			(at 151.384 161.036 90)
 			(hide yes)
@@
 			)
 		)
-		(property "Footprint" "Resistor_SMD:R_0805_2012Metric_Pad1.20x1.40mm_HandSolder"
+		(property "Footprint" "Resistor_SMD:R_0603_1608Metric_Pad0.98x0.95mm_HandSolder"
 			(at 151.384 35.306 90)
 			(hide yes)
@@
 			)
 		)
-		(property "Footprint" "Resistor_SMD:R_0805_2012Metric_Pad1.20x1.40mm_HandSolder"
+		(property "Footprint" "Resistor_SMD:R_0603_1608Metric_Pad0.98x0.95mm_HandSolder"
 			(at 151.384 105.156 90)
 			(hide yes)
